Commit message: Added simulated hokuyo lidar.

File: src/turtlebot_description/robots/kobuki_hexagons_asus_xtion_pro.urdf.xacro (robot description, xacro)
@@ -10,4 +10,8 @@
   <xacro:include filename="$(find turtlebot_description)/urdf/stacks/hexagons.urdf.xacro"/>
   <xacro:include filename="$(find turtlebot_description)/urdf/sensors/asus_xtion_pro.urdf.xacro"/>
+  <xacro:include filename="$(find hector_sensors_description)/urdf/hokuyo_utm30lx.urdf.xacro" />
+  <xacro:hokuyo_utm30lx name="hokuyo_laser" parent="base_link" ros_topic="hokuyo_scan" update_rate="40" ray_count="1040" min_angle="130" max_angle="-130">
+    <origin xyz="0.0925 -0.004 0.198" rpy="0 0 0"/>
+  </xacro:hokuyo_utm30lx>
   <kobuki/>
   <stack_hexagons                 parent="base_link"/>

Commit message: Changed from Hokuyo to rplidar.

File: src/turtlebot_description/robots/kobuki_hexagons_asus_xtion_pro.urdf.xacro (robot description, xacro)
@@ -6,14 +6,12 @@
 -->
 <robot name="turtlebot" xmlns:xacro="http://ros.org/wiki/xacro">
-  <xacro:include filename="$(find turtlebot_description)/urdf/turtlebot_common_library.urdf.xacro" />
-  <xacro:include filename="$(find kobuki_description)/urdf/kobuki.urdf.xacro" />
+  <xacro:include filename="$(find turtlebot_description)/urdf/turtlebot_common_library.urdf.xacro"/>
+  <xacro:include filename="$(find kobuki_description)/urdf/kobuki.urdf.xacro"/>
   <xacro:include filename="$(find turtlebot_description)/urdf/stacks/hexagons.urdf.xacro"/>
   <!--<xacro:include filename="$(find turtlebot_description)/urdf/sensors/asus_xtion_pro.urdf.xacro"/>-->
-  <xacro:include filename="$(find turtlebot_description)/urdf/sensors/hokuyo_utm30lx.urdf.xacro" />
-  <xacro:hokuyo_utm30lx name="hokuyo_laser" parent="base_link" ros_topic="scan" update_rate="5.5" ray_count="2000" min_angle="0" max_angle="360">
-    <origin xyz="0.0925 -0.004 0.198" rpy="0 0 0"/>
-  </xacro:hokuyo_utm30lx>
+  <xacro:include filename="$(find turtlebot_description)/urdf/sensors/rplidar.urdf.xacro"/>
   <kobuki/>
-  <stack_hexagons                 parent="base_link"/>
-  <sensor_asus_xtion_pro          parent="base_link"/>
+  <stack_hexagons parent="base_link"/>
+  <!--<sensor_asus_xtion_pro          parent="base_link"/>-->
+  <sensor_rplidar parent="plate_middle_link" ros_topic="scan" name="rplidar"/>
 </robot>
